File: hw/sch_pcb/CPU.kicad_sch (KiCad schematic)
At the start: 48 parts, among them J1 SM06B-GHS-TB, J4 HEADER_2x03, J5 SM08B-GHS-TB, J6 SM06B-GHS-TB, SW1 KMT031 NGJ LHS C&K, U7 SHT31, U8 ATMEGA1284P-AU, U9 AT24CS64-SSHM, Y1 16MHz

Commit message: Editing component values
Parts:
- C25: UST_ID (none) -> 5e3ff54b1287502a33bad705
Changed lines of the file:
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@@
+      (effects (font (size 1.27 1.27)) hide)
+    )
+    (property "UST_ID" "5e3ff54b1287502a33bad705" (at 255.27 146.05 0)
       (effects (font (size 1.27 1.27)) hide)
     )

Commit message: Updated title block.
Other:
- company: (none) -> ust.cz
- title: (none) -> THUNDERMILL01B
Changed lines of the file:
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@@
 (kicad_sch (version 20230121) (generator eeschema)
   (paper "A4")
+  (title_block
+    (title "THUNDERMILL01B")
+    (company "ust.cz")
+    (comment 1 "Stator PCB\\n - signal processing board")
+  )
   (junction (at 227.33 72.39) (diameter 1.016) (color 0 0 0 0)
   )
