File: hw/sch_pcb/USTTHUNDERMILLPCB01.kicad_sch (KiCad schematic)
At the start: 15 parts, among them J2 SM03B-GHS-TB, J3 HEADER_1x01, U1 ISL21080DIH312Z-TK 1V25, U2 OPA314

Commit message: Updated title block.
Other:
- company: (none) -> ust.cz
- title: (none) -> THUNDERMILL01B
Changed lines of the file:
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@@
 (kicad_sch (version 20230121) (generator eeschema)
   (paper "A4")
+  (title_block
+    (title "THUNDERMILL01B")
+    (date "2023-11-04")
+    (company "ust.cz")
+    (comment 1 "Stator PCB\\n - signal processing board")
+  )
   (junction (at 106.68 78.74) (diameter 1.016) (color 0 0 0 0)
   )
