File: hw/sch_pcb/tachometer.kicad_sch (KiCad schematic)
At the start: 24 parts, among them U10 SN74LVC1G14QDCKRQ1, U11 SN74LVC1G14QDCKRQ1, U12 SN74LVC1G14QDCKRQ1, U13 VCNT2020, U3 MIC5504-3.3YM5, U4 PCF8583, U5 VCNT2020, U6 VCNT2020

Commit message: Editing component values
Parts:
- F1: UST_ID (none) -> 5c70984512875079b91f88d1
Changed lines of the file:
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@@
+      (effects (font (size 1.27 1.27)) hide)
+    )
+    (property "UST_ID" "5c70984512875079b91f88d1" (at 24.13 165.1 0)
       (effects (font (size 1.27 1.27)) hide)
     )

Commit message: Updated title block.
Other:
- company: (none) -> ust.cz
- title: (none) -> THUNDERMILL01B
Changed lines of the file:
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@@
 (kicad_sch (version 20230121) (generator eeschema)
   (paper "A4")
+  (title_block
+    (title "THUNDERMILL01B")
+    (company "ust.cz")
+    (comment 1 "Stator PCB\\n - signal processing board")
+  )
   (junction (at 27.94 172.72) (diameter 0) (color 0 0 0 0)
   )
